Commit message: optimize foot concat with ground

File: assets/ths_t1/urdf/ths_t1.urdf (robot description, URDF)
Before this commit: robot ths_t3_tpos_urdf, 26 links, 25 joints
Links:
- added link left_leg_heel_link
- added link left_leg_toe_link
- added link right_leg_heel_link
- added link right_leg_toe_link
Joints:
- added joint left_leg_heel_joint: type fixed, parent left_leg_ankle_link, child left_leg_heel_link, origin xyz=-0.05 0 -0.05 rpy=0 0 0
- added joint left_leg_toe_joint: type fixed, parent left_leg_ankle_link, child left_leg_toe_link, origin xyz=0.13 0 -0.05 rpy=0 0 0
- added joint right_leg_heel_joint: type fixed, parent right_leg_ankle_link, child right_leg_heel_link, origin xyz=-0.05 0 -0.05 rpy=0 0 0
- added joint right_leg_toe_joint: type fixed, parent right_leg_ankle_link, child right_leg_toe_link, origin xyz=0.13 0 -0.05 rpy=0 0 0
